File: bepocious/bepocious.sch (KiCad schematic (older format))
At the start: 14 parts

Commit message: No changes
Parts:
- U?: symbol MCU_Microchip_ATmega:ATmega32U4-MU -> bepocious-rescue:ATmega32U4-MU-MCU_Microchip_ATmega
Changed lines of the file:
@@
 EESchema Schematic File Version 4
+LIBS:bepocious-cache
 EELAYER 30 0
 EELAYER END
@@
 $EndDescr
 $Comp
-L MCU_Microchip_ATmega:ATmega32U4-MU U?
+L bepocious-rescue:ATmega32U4-MU-MCU_Microchip_ATmega U?
 U 1 1 6041EC71
 P 7450 3650
